Commit message: add zq robot

File: legged_gym/resources/robots/zq_humanoid/urdf/zq_sa01.urdf (robot description, URDF)
Before this commit: robot zqsa01, 13 links, 12 joints
Links:
- added link keyframe_head_link; visual box size=0.01 0.01 0.01
Joints:
- added joint keyframe_head_joint: type fixed, parent base_link, child keyframe_head_link, origin xyz=0 0 0.08 rpy=0 0 0

Commit message: zq urdf

File: legged_gym/resources/robots/zq_humanoid/urdf/zq_sa01.urdf (robot description, URDF)
Before this commit: robot zqsa01, 14 links, 13 joints
Links:
- added link auxiliary_l_ankle_roll_link1; visual sphere radius=0.01
- added link auxiliary_l_ankle_roll_link2; visual sphere radius=0.01
- added link auxiliary_l_ankle_roll_link3; visual sphere radius=0.01
- added link auxiliary_l_ankle_roll_link4; visual sphere radius=0.01
- added link auxiliary_r_ankle_roll_link1; visual sphere radius=0.01
- added link auxiliary_r_ankle_roll_link2; visual sphere radius=0.01
- added link auxiliary_r_ankle_roll_link3; visual sphere radius=0.01
- added link auxiliary_r_ankle_roll_link4; visual sphere radius=0.01
- link leg_l6_link: geometry collision mesh filename=../meshes/LeftLeg_Link_06.STL; collision sphere radius=0.005
- link leg_r6_link: geometry collision mesh filename=../meshes/RightLeg_Link_06.STL; collision sphere radius=0.005
Joints:
- added joint auxiliary_l_ankle_roll_joint1: type fixed, parent leg_l6_link, child auxiliary_l_ankle_roll_link1, origin xyz=0.05 -0.07 -0.045 rpy=0 0 0
- added joint auxiliary_l_ankle_roll_joint2: type fixed, parent leg_l6_link, child auxiliary_l_ankle_roll_link2, origin xyz=0.05 0.08 -0.045 rpy=0 0 0
- added joint auxiliary_l_ankle_roll_joint3: type fixed, parent leg_l6_link, child auxiliary_l_ankle_roll_link3, origin xyz=0.23 0 -0.045 rpy=0 0 0
- added joint auxiliary_l_ankle_roll_joint4: type fixed, parent leg_l6_link, child auxiliary_l_ankle_roll_link4, origin xyz=-0.11 0 -0.045 rpy=0 0 0
- added joint auxiliary_r_ankle_roll_joint1: type fixed, parent leg_r6_link, child auxiliary_r_ankle_roll_link1, origin xyz=0.05 -0.08 -0.045 rpy=0 0 0
- added joint auxiliary_r_ankle_roll_joint2: type fixed, parent leg_r6_link, child auxiliary_r_ankle_roll_link2, origin xyz=0.05 0.07 -0.045 rpy=0 0 0
- added joint auxiliary_r_ankle_roll_joint3: type fixed, parent leg_r6_link, child auxiliary_r_ankle_roll_link3, origin xyz=0.23 0 -0.045 rpy=0 0 0
- added joint auxiliary_r_ankle_roll_joint4: type fixed, parent leg_r6_link, child auxiliary_r_ankle_roll_link4, origin xyz=-0.11 0 -0.045 rpy=0 0 0
- joint keyframe_head_joint: origin xyz=0 0 0.08 rpy=0 0 0 -> xyz=0 0 0.4 rpy=0 0 0
